File: MiniSplit.sch (KiCad schematic (older format))
At the start: 49 parts, among them J1 5PIN, SW1 SW_PUSH, SW10 SW_PUSH, SW11 SW_PUSH, SW12 SW_PUSH, SW13 SW_PUSH, SW14 SW_PUSH, SW15 SW_PUSH, SW16 SW_PUSH, SW17 SW_PUSH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

Commit message: fix #1 #2
Parts:
- SW1, SW10, SW11, SW12, SW13, SW14, SW15, SW16, SW17, SW18, SW19, SW2, SW20, SW21, SW3, SW4, SW5, SW6, SW7, SW8, SW9: footprint minisplit-footprint:MX_FLIP_HOLES -> lets_split-footprint:MXALPS_FLIP_HOLES
Changed lines of the file:
@@
 LIBS:lets_split-cache
 LIBS:local
+LIBS:promicro
 LIBS:ir2153
 LIBS:irf7103
@@
 F 0 "SW2" H 6900 3510 50  0000 C CNN
 F 1 "SW_PUSH" H 6750 3320 50  0000 C CNN
-F 2 "minisplit-footprint:MX_FLIP_HOLES" H 6750 3400 50  0001 C CNN
+F 2 "lets_split-footprint:MXALPS_FLIP_HOLES" H 6750 3400 50  0001 C CNN
 F 3 "" H 6750 3400 50  0000 C CNN
 	1    6750 3400
@@
 F 0 "SW7" H 7650 4010 50  0000 C CNN
 F 1 "SW_PUSH" H 7500 3820 50  0000 C CNN
-F 2 "minisplit-footprint:MX_FLIP_HOLES" H 7500 3900 50  0001 C CNN
+F 2 "lets_split-footprint:MXALPS_FLIP_HOLES" H 7500 3900 50  0001 C CNN
 F 3 "" H 7500 3900 50  0000 C CNN
 	1    7500 3900
@@
 F 0 "SW11" H 8400 4010 50  0000 C CNN
 F 1 "SW_PUSH" H 8250 3820 50  0000 C CNN
-F 2 "minisplit-footprint:MX_FLIP_HOLES" H 8250 3900 50  0001 C CNN
+F 2 "lets_split-footprint:MXALPS_FLIP_HOLES" H 8250 3900 50  0001 C CNN
 F 3 "" H 8250 3900 50  0000 C CNN
 	1    8250 3900
@@
 F 0 "SW3" H 6900 4010 50  0000 C CNN
 F 1 "SW_PUSH" H 6750 3820 50  0000 C CNN
-F 2 "minisplit-footprint:MX_FLIP_HOLES" H 6750 3900 50  0001 C CNN
+F 2 "lets_split-footprint:MXALPS_FLIP_HOLES" H 6750 3900 50  0001 C CNN
 F 3 "" H 6750 3900 50  0000 C CNN
 	1    6750 3900
@@
 F 0 "SW17" H 9900 4010 50  0000 C CNN
 F 1 "SW_PUSH" H 9750 3820 50  0000 C CNN
-F 2 "minisplit-footprint:MX_FLIP_HOLES" H 9750 3900 50  0001 C CNN
+F 2 "lets_split-footprint:MXALPS_FLIP_HOLES" H 9750 3900 50  0001 C CNN
 F 3 "" H 9750 3900 50  0000 C CNN
 	1    9750 3900
@@
 F 0 "SW20" H 10650 4010 50  0000 C CNN
 F 1 "SW_PUSH" H 10500 3820 50  0000 C CNN
-F 2 "minisplit-footprint:MX_FLIP_HOLES" H 10500 3900 50  0001 C CNN
+F 2 "lets_split-footprint:MXALPS_FLIP_HOLES" H 10500 3900 50  0001 C CNN
 F 3 "" H 10500 3900 50  0000 C CNN
 	1    10500 3900
@@
 F 0 "SW14" H 9150 4010 50  0000 C CNN
 F 1 "SW_PUSH" H 9000 3820 50  0000 C CNN
-F 2 "minisplit-footprint:MX_FLIP_HOLES" H 9000 3900 50  0001 C CNN
+F 2 "lets_split-footprint:MXALPS_FLIP_HOLES" H 9000 3900 50  0001 C CNN
 F 3 "" H 9000 3900 50  0000 C CNN
 	1    9000 3900
@@
 F 0 "SW8" H 7650 4510 50  0000 C CNN
 F 1 "SW_PUSH" H 7500 4320 50  0000 C CNN
-F 2 "minisplit-footprint:MX_FLIP_HOLES" H 7500 4400 50  0001 C CNN
+F 2 "lets_split-footprint:MXALPS_FLIP_HOLES" H 7500 4400 50  0001 C CNN
 F 3 "" H 7500 4400 50  0000 C CNN
 	1    7500 4400
@@
 F 0 "SW12" H 8400 4510 50  0000 C CNN
 F 1 "SW_PUSH" H 8250 4320 50  0000 C CNN
-F 2 "minisplit-footprint:MX_FLIP_HOLES" H 8250 4400 50  0001 C CNN
+F 2 "lets_split-footprint:MXALPS_FLIP_HOLES" H 8250 4400 50  0001 C CNN
 F 3 "" H 8250 4400 50  0000 C CNN
 	1    8250 4400
@@
 F 0 "SW4" H 6900 4510 50  0000 C CNN
 F 1 "SW_PUSH" H 6750 4320 50  0000 C CNN
-F 2 "minisplit-footprint:MX_FLIP_HOLES" H 6750 4400 50  0001 C CNN
+F 2 "lets_split-footprint:MXALPS_FLIP_HOLES" H 6750 4400 50  0001 C CNN
 F 3 "" H 6750 4400 50  0000 C CNN
 	1    6750 4400
@@
 F 0 "SW18" H 9900 4510 50  0000 C CNN
 F 1 "SW_PUSH" H 9750 4320 50  0000 C CNN
-F 2 "minisplit-footprint:MX_FLIP_HOLES" H 9750 4400 50  0001 C CNN
+F 2 "lets_split-footprint:MXALPS_FLIP_HOLES" H 9750 4400 50  0001 C CNN
 F 3 "" H 9750 4400 50  0000 C CNN
 	1    9750 4400
@@
 F 0 "SW21" H 10650 4510 50  0000 C CNN
 F 1 "SW_PUSH" H 10500 4320 50  0000 C CNN
-F 2 "minisplit-footprint:MX_FLIP_HOLES" H 10500 4400 50  0001 C CNN
+F 2 "lets_split-footprint:MXALPS_FLIP_HOLES" H 10500 4400 50  0001 C CNN
 F 3 "" H 10500 4400 50  0000 C CNN
 	1    10500 4400
@@
 F 0 "SW15" H 9150 4510 50  0000 C CNN
 F 1 "SW_PUSH" H 9000 4320 50  0000 C CNN
-F 2 "minisplit-footprint:MX_FLIP_HOLES" H 9000 4400 50  0001 C CNN
+F 2 "lets_split-footprint:MXALPS_FLIP_HOLES" H 9000 4400 50  0001 C CNN
 F 3 "" H 9000 4400 50  0000 C CNN
 	1    9000 4400
@@
 F 0 "SW5" H 6900 5010 50  0000 C CNN
 F 1 "SW_PUSH" H 6750 4820 50  0000 C CNN
-F 2 "minisplit-footprint:MX_FLIP_HOLES" H 6750 4900 50  0001 C CNN
+F 2 "lets_split-footprint:MXALPS_FLIP_HOLES" H 6750 4900 50  0001 C CNN
 F 3 "" H 6750 4900 50  0000 C CNN
 	1    6750 4900
@@
 F 0 "SW9" H 7650 5010 50  0000 C CNN
 F 1 "SW_PUSH" H 7500 4820 50  0000 C CNN
-F 2 "minisplit-footprint:MX_FLIP_HOLES" H 7500 4900 50  0001 C CNN
+F 2 "lets_split-footprint:MXALPS_FLIP_HOLES" H 7500 4900 50  0001 C CNN
 F 3 "" H 7500 4900 50  0000 C CNN
 	1    7500 4900
@@
 F 0 "SW1" H 6150 5010 50  0000 C CNN
 F 1 "SW_PUSH" H 6000 4820 50  0000 C CNN
-F 2 "minisplit-footprint:MX_FLIP_HOLES" H 6000 4900 50  0001 C CNN
+F 2 "lets_split-footprint:MXALPS_FLIP_HOLES" H 6000 4900 50  0001 C CNN
 F 3 "" H 6000 4900 50  0000 C CNN
 	1    6000 4900
@@
 F 0 "SW6" H 7650 3510 50  0000 C CNN
 F 1 "SW_PUSH" H 7500 3320 50  0000 C CNN
-F 2 "minisplit-footprint:MX_FLIP_HOLES" H 7500 3400 50  0001 C CNN
+F 2 "lets_split-footprint:MXALPS_FLIP_HOLES" H 7500 3400 50  0001 C CNN
 F 3 "" H 7500 3400 50  0000 C CNN
 	1    7500 3400
@@
 F 0 "SW10" H 8400 3510 50  0000 C CNN
 F 1 "SW_PUSH" H 8250 3320 50  0000 C CNN
-F 2 "minisplit-footprint:MX_FLIP_HOLES" H 8250 3400 50  0001 C CNN
+F 2 "lets_split-footprint:MXALPS_FLIP_HOLES" H 8250 3400 50  0001 C CNN
 F 3 "" H 8250 3400 50  0000 C CNN
 	1    8250 3400
@@
 F 0 "SW16" H 9900 3510 50  0000 C CNN
 F 1 "SW_PUSH" H 9750 3320 50  0000 C CNN
-F 2 "minisplit-footprint:MX_FLIP_HOLES" H 9750 3400 50  0001 C CNN
+F 2 "lets_split-footprint:MXALPS_FLIP_HOLES" H 9750 3400 50  0001 C CNN
 F 3 "" H 9750 3400 50  0000 C CNN
 	1    9750 3400
@@
 F 0 "SW19" H 10650 3510 50  0000 C CNN
 F 1 "SW_PUSH" H 10500 3320 50  0000 C CNN
-F 2 "minisplit-footprint:MX_FLIP_HOLES" H 10500 3400 50  0001 C CNN
+F 2 "lets_split-footprint:MXALPS_FLIP_HOLES" H 10500 3400 50  0001 C CNN
 F 3 "" H 10500 3400 50  0000 C CNN
 	1    10500 3400
@@
 F 0 "SW13" H 9150 3510 50  0000 C CNN
 F 1 "SW_PUSH" H 9000 3320 50  0000 C CNN
-F 2 "minisplit-footprint:MX_FLIP_HOLES" H 9000 3400 50  0001 C CNN
+F 2 "lets_split-footprint:MXALPS_FLIP_HOLES" H 9000 3400 50  0001 C CNN
 F 3 "" H 9000 3400 50  0000 C CNN
 	1    9000 3400

Commit message: fix file
Parts:
- SW1, SW10, SW11, SW12, SW13, SW14, SW15, SW16, SW17, SW18, SW19, SW2, SW20, SW21, SW3, SW4, SW5, SW6, SW7, SW8, SW9: footprint lets_split-footprint:MXALPS_FLIP_HOLES -> minisplit-footprint:MX_FLIP_HOLES
Changed lines of the file:
@@
 LIBS:lets_split-cache
 LIBS:local
-LIBS:promicro
 LIBS:ir2153
 LIBS:irf7103
@@
 F 0 "SW2" H 6900 3510 50  0000 C CNN
 F 1 "SW_PUSH" H 6750 3320 50  0000 C CNN
-F 2 "lets_split-footprint:MXALPS_FLIP_HOLES" H 6750 3400 50  0001 C CNN
+F 2 "minisplit-footprint:MX_FLIP_HOLES" H 6750 3400 50  0001 C CNN
 F 3 "" H 6750 3400 50  0000 C CNN
 	1    6750 3400
@@
 F 0 "SW7" H 7650 4010 50  0000 C CNN
 F 1 "SW_PUSH" H 7500 3820 50  0000 C CNN
-F 2 "lets_split-footprint:MXALPS_FLIP_HOLES" H 7500 3900 50  0001 C CNN
+F 2 "minisplit-footprint:MX_FLIP_HOLES" H 7500 3900 50  0001 C CNN
 F 3 "" H 7500 3900 50  0000 C CNN
 	1    7500 3900
@@
 F 0 "SW11" H 8400 4010 50  0000 C CNN
 F 1 "SW_PUSH" H 8250 3820 50  0000 C CNN
-F 2 "lets_split-footprint:MXALPS_FLIP_HOLES" H 8250 3900 50  0001 C CNN
+F 2 "minisplit-footprint:MX_FLIP_HOLES" H 8250 3900 50  0001 C CNN
 F 3 "" H 8250 3900 50  0000 C CNN
 	1    8250 3900
@@
 F 0 "SW3" H 6900 4010 50  0000 C CNN
 F 1 "SW_PUSH" H 6750 3820 50  0000 C CNN
-F 2 "lets_split-footprint:MXALPS_FLIP_HOLES" H 6750 3900 50  0001 C CNN
+F 2 "minisplit-footprint:MX_FLIP_HOLES" H 6750 3900 50  0001 C CNN
 F 3 "" H 6750 3900 50  0000 C CNN
 	1    6750 3900
@@
 F 0 "SW17" H 9900 4010 50  0000 C CNN
 F 1 "SW_PUSH" H 9750 3820 50  0000 C CNN
-F 2 "lets_split-footprint:MXALPS_FLIP_HOLES" H 9750 3900 50  0001 C CNN
+F 2 "minisplit-footprint:MX_FLIP_HOLES" H 9750 3900 50  0001 C CNN
 F 3 "" H 9750 3900 50  0000 C CNN
 	1    9750 3900
@@
 F 0 "SW20" H 10650 4010 50  0000 C CNN
 F 1 "SW_PUSH" H 10500 3820 50  0000 C CNN
-F 2 "lets_split-footprint:MXALPS_FLIP_HOLES" H 10500 3900 50  0001 C CNN
+F 2 "minisplit-footprint:MX_FLIP_HOLES" H 10500 3900 50  0001 C CNN
 F 3 "" H 10500 3900 50  0000 C CNN
 	1    10500 3900
@@
 F 0 "SW14" H 9150 4010 50  0000 C CNN
 F 1 "SW_PUSH" H 9000 3820 50  0000 C CNN
-F 2 "lets_split-footprint:MXALPS_FLIP_HOLES" H 9000 3900 50  0001 C CNN
+F 2 "minisplit-footprint:MX_FLIP_HOLES" H 9000 3900 50  0001 C CNN
 F 3 "" H 9000 3900 50  0000 C CNN
 	1    9000 3900
@@
 F 0 "SW8" H 7650 4510 50  0000 C CNN
 F 1 "SW_PUSH" H 7500 4320 50  0000 C CNN
-F 2 "lets_split-footprint:MXALPS_FLIP_HOLES" H 7500 4400 50  0001 C CNN
+F 2 "minisplit-footprint:MX_FLIP_HOLES" H 7500 4400 50  0001 C CNN
 F 3 "" H 7500 4400 50  0000 C CNN
 	1    7500 4400
@@
 F 0 "SW12" H 8400 4510 50  0000 C CNN
 F 1 "SW_PUSH" H 8250 4320 50  0000 C CNN
-F 2 "lets_split-footprint:MXALPS_FLIP_HOLES" H 8250 4400 50  0001 C CNN
+F 2 "minisplit-footprint:MX_FLIP_HOLES" H 8250 4400 50  0001 C CNN
 F 3 "" H 8250 4400 50  0000 C CNN
 	1    8250 4400
@@
 F 0 "SW4" H 6900 4510 50  0000 C CNN
 F 1 "SW_PUSH" H 6750 4320 50  0000 C CNN
-F 2 "lets_split-footprint:MXALPS_FLIP_HOLES" H 6750 4400 50  0001 C CNN
+F 2 "minisplit-footprint:MX_FLIP_HOLES" H 6750 4400 50  0001 C CNN
 F 3 "" H 6750 4400 50  0000 C CNN
 	1    6750 4400
@@
 F 0 "SW18" H 9900 4510 50  0000 C CNN
 F 1 "SW_PUSH" H 9750 4320 50  0000 C CNN
-F 2 "lets_split-footprint:MXALPS_FLIP_HOLES" H 9750 4400 50  0001 C CNN
+F 2 "minisplit-footprint:MX_FLIP_HOLES" H 9750 4400 50  0001 C CNN
 F 3 "" H 9750 4400 50  0000 C CNN
 	1    9750 4400
@@
 F 0 "SW21" H 10650 4510 50  0000 C CNN
 F 1 "SW_PUSH" H 10500 4320 50  0000 C CNN
-F 2 "lets_split-footprint:MXALPS_FLIP_HOLES" H 10500 4400 50  0001 C CNN
+F 2 "minisplit-footprint:MX_FLIP_HOLES" H 10500 4400 50  0001 C CNN
 F 3 "" H 10500 4400 50  0000 C CNN
 	1    10500 4400
@@
 F 0 "SW15" H 9150 4510 50  0000 C CNN
 F 1 "SW_PUSH" H 9000 4320 50  0000 C CNN
-F 2 "lets_split-footprint:MXALPS_FLIP_HOLES" H 9000 4400 50  0001 C CNN
+F 2 "minisplit-footprint:MX_FLIP_HOLES" H 9000 4400 50  0001 C CNN
 F 3 "" H 9000 4400 50  0000 C CNN
 	1    9000 4400
@@
 F 0 "SW5" H 6900 5010 50  0000 C CNN
 F 1 "SW_PUSH" H 6750 4820 50  0000 C CNN
-F 2 "lets_split-footprint:MXALPS_FLIP_HOLES" H 6750 4900 50  0001 C CNN
+F 2 "minisplit-footprint:MX_FLIP_HOLES" H 6750 4900 50  0001 C CNN
 F 3 "" H 6750 4900 50  0000 C CNN
 	1    6750 4900
@@
 F 0 "SW9" H 7650 5010 50  0000 C CNN
 F 1 "SW_PUSH" H 7500 4820 50  0000 C CNN
-F 2 "lets_split-footprint:MXALPS_FLIP_HOLES" H 7500 4900 50  0001 C CNN
+F 2 "minisplit-footprint:MX_FLIP_HOLES" H 7500 4900 50  0001 C CNN
 F 3 "" H 7500 4900 50  0000 C CNN
 	1    7500 4900
@@
 F 0 "SW1" H 6150 5010 50  0000 C CNN
 F 1 "SW_PUSH" H 6000 4820 50  0000 C CNN
-F 2 "lets_split-footprint:MXALPS_FLIP_HOLES" H 6000 4900 50  0001 C CNN
+F 2 "minisplit-footprint:MX_FLIP_HOLES" H 6000 4900 50  0001 C CNN
 F 3 "" H 6000 4900 50  0000 C CNN
 	1    6000 4900
@@
 F 0 "SW6" H 7650 3510 50  0000 C CNN
 F 1 "SW_PUSH" H 7500 3320 50  0000 C CNN
-F 2 "lets_split-footprint:MXALPS_FLIP_HOLES" H 7500 3400 50  0001 C CNN
+F 2 "minisplit-footprint:MX_FLIP_HOLES" H 7500 3400 50  0001 C CNN
 F 3 "" H 7500 3400 50  0000 C CNN
 	1    7500 3400
@@
 F 0 "SW10" H 8400 3510 50  0000 C CNN
 F 1 "SW_PUSH" H 8250 3320 50  0000 C CNN
-F 2 "lets_split-footprint:MXALPS_FLIP_HOLES" H 8250 3400 50  0001 C CNN
+F 2 "minisplit-footprint:MX_FLIP_HOLES" H 8250 3400 50  0001 C CNN
 F 3 "" H 8250 3400 50  0000 C CNN
 	1    8250 3400
@@
 F 0 "SW16" H 9900 3510 50  0000 C CNN
 F 1 "SW_PUSH" H 9750 3320 50  0000 C CNN
-F 2 "lets_split-footprint:MXALPS_FLIP_HOLES" H 9750 3400 50  0001 C CNN
+F 2 "minisplit-footprint:MX_FLIP_HOLES" H 9750 3400 50  0001 C CNN
 F 3 "" H 9750 3400 50  0000 C CNN
 	1    9750 3400
@@
 F 0 "SW19" H 10650 3510 50  0000 C CNN
 F 1 "SW_PUSH" H 10500 3320 50  0000 C CNN
-F 2 "lets_split-footprint:MXALPS_FLIP_HOLES" H 10500 3400 50  0001 C CNN
+F 2 "minisplit-footprint:MX_FLIP_HOLES" H 10500 3400 50  0001 C CNN
 F 3 "" H 10500 3400 50  0000 C CNN
 	1    10500 3400
@@
 F 0 "SW13" H 9150 3510 50  0000 C CNN
 F 1 "SW_PUSH" H 9000 3320 50  0000 C CNN
-F 2 "lets_split-footprint:MXALPS_FLIP_HOLES" H 9000 3400 50  0001 C CNN
+F 2 "minisplit-footprint:MX_FLIP_HOLES" H 9000 3400 50  0001 C CNN
 F 3 "" H 9000 3400 50  0000 C CNN
 	1    9000 3400
